File: kicad/electret_preamp.sch (KiCad schematic (older format))
At the start: 16 parts, among them U1 NE5532

Commit message: Fix errors in KiCAD files
Parts:
- C6: footprint (none) -> Capacitor_SMD:CP_Elec_4x5.8; symbol Device:C -> Device:CP
- R2: value 270k -> 180k
Connections:
- net at C2.2, C3.2, R2.2: now also U1.2 (-); no longer U1.3 (+)
- net at C6.1, R3.2, R5.1: now also U1.3 (+); no longer U1.2 (-)
Changed lines of the file:
@@
 EESchema Schematic File Version 4
+LIBS:electret_preamp-cache
 EELAYER 29 0
 EELAYER END
@@
 P 2400 1500
 F 0 "R2" V 2193 1500 50  0000 C CNN
-F 1 "270k" V 2284 1500 50  0000 C CNN
+F 1 "180k" V 2284 1500 50  0000 C CNN
 F 2 "Resistor_SMD:R_1210_3225Metric_Pad1.42x2.65mm_HandSolder" V 2330 1500 50  0001 C CNN
 F 3 "~" H 2400 1500 50  0001 C CNN
@@
 $EndComp
 $Comp
-L Device:C C6
+L Device:CP C6
 U 1 1 5ED1A83D
 P 1950 3100
 F 0 "C6" H 2065 3146 50  0000 L CNN
 F 1 "10u" H 2065 3055 50  0000 L CNN
-F 2 "" H 1988 2950 50  0001 C CNN
+F 2 "Capacitor_SMD:CP_Elec_4x5.8" H 1988 2950 50  0001 C CNN
 F 3 "~" H 1950 3100 50  0001 C CNN
 	1    1950 3100
@@
 F 3 "http://www.ti.com/lit/ds/symlink/ne5532.pdf" H 2350 2050 50  0001 C CNN
 	1    2350 2050
-	1    0    0    -1
-$EndComp
-$Comp
+	1    0    0    1
+$EndComp
+$Comp

Commit message: Polarized cap in wrong direction
Parts:
- C4: symbol Device:C -> Device:CP
Connections:
- net +5V: now also C4.1; no longer C4.2
- net GND: now also C4.2; no longer C4.1
Changed lines of the file:
@@
 $EndComp
 $Comp
-L Device:C C4
+L Device:CP C4
 U 1 1 5ED3F871
 P 4450 4500
-F 0 "C4" H 4335 4454 50  0000 R CNN
-F 1 "10u" H 4335 4545 50  0000 R CNN
+F 0 "C4" H 4700 4550 50  0000 R CNN
+F 1 "10u" H 4700 4450 50  0000 R CNN
 F 2 "Capacitor_SMD:CP_Elec_6.3x9.9" H 4488 4350 50  0001 C CNN
 F 3 "~" H 4450 4500 50  0001 C CNN
 	1    4450 4500
-	-1   0    0    1
+	1    0    0    -1
 $EndComp
 Wire Wire Line
